File: MinimumKeyboard/MinimumKeyboard.kicad_sch (KiCad schematic)
At the start: 12 parts, among them J1 MJ-4PP-9, J2 LED, SW1 SW_PUSH, SW2 SW_PUSH, SW3 SW_PUSH, SW4 SW_PUSH, SW5 SW_PUSH, U1 ProMicro

Commit message: footprint assignment
Parts:
- D1, D2, D3, D4: footprint (none) -> kbd.pretty:D3_SMD
- J1: footprint (none) -> kbd.pretty:MJ-4PP-9
- J2: footprint kbd:StripLED_rev -> kbd.pretty:StripLED_rev
- SW1, SW2, SW3, SW4, SW5: footprint (none) -> kbd.pretty:CherryMX_Choc_Hotswap
- U1: footprint (none) -> kbd.pretty:ProMicro_v2
Changed lines of the file:
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@@
     (property "Reference" "SW4" (id 0) (at 124.46 121.92 0))
     (property "Value" "SW_PUSH" (id 1) (at 124.46 124.46 0))
-    (property "Footprint" "" (id 2) (at 124.46 129.54 0))
+    (property "Footprint" "kbd.pretty:CherryMX_Choc_Hotswap" (id 2) (at 124.46 129.54 0)
+      (effects (font (size 1.27 1.27)) hide)
+    )
     (property "Datasheet" "" (id 3) (at 124.46 129.54 0))
     (pin "1")
@@
     (property "Reference" "SW1" (id 0) (at 87.63 100.33 0))
     (property "Value" "SW_PUSH" (id 1) (at 87.63 102.87 0))
-    (property "Footprint" "" (id 2) (at 87.63 107.95 0))
+    (property "Footprint" "kbd.pretty:CherryMX_Choc_Hotswap" (id 2) (at 87.63 107.95 0)
+      (effects (font (size 1.27 1.27)) hide)
+    )
     (property "Datasheet" "" (id 3) (at 87.63 107.95 0))
     (pin "1")
@@
     (property "Reference" "J1" (id 0) (at 37.7825 69.85 0))
     (property "Value" "MJ-4PP-9" (id 1) (at 37.7825 72.39 0))
-    (property "Footprint" "" (id 2) (at 45.085 73.025 0)
+    (property "Footprint" "kbd.pretty:MJ-4PP-9" (id 2) (at 45.085 73.025 0)
       (effects (font (size 1.27 1.27)) hide)
     )
@@
       (effects (font (size 1.27 1.27)) (justify right))
     )
-    (property "Footprint" "" (id 2) (at 132.08 133.35 0)
+    (property "Footprint" "kbd.pretty:D3_SMD" (id 2) (at 132.08 133.35 0)
       (effects (font (size 1.27 1.27)) hide)
     )
@@
     (property "Reference" "SW3" (id 0) (at 124.46 100.33 0))
     (property "Value" "SW_PUSH" (id 1) (at 124.46 102.87 0))
-    (property "Footprint" "" (id 2) (at 124.46 107.95 0))
+    (property "Footprint" "kbd.pretty:CherryMX_Choc_Hotswap" (id 2) (at 124.46 107.95 0)
+      (effects (font (size 1.27 1.27)) hide)
+    )
     (property "Datasheet" "" (id 3) (at 124.46 107.95 0))
     (pin "1")
@@
     (property "Reference" "SW2" (id 0) (at 87.63 121.92 0))
     (property "Value" "SW_PUSH" (id 1) (at 87.63 124.46 0))
-    (property "Footprint" "" (id 2) (at 87.63 129.54 0))
+    (property "Footprint" "kbd.pretty:CherryMX_Choc_Hotswap" (id 2) (at 87.63 129.54 0)
+      (effects (font (size 1.27 1.27)) hide)
+    )
     (property "Datasheet" "" (id 3) (at 87.63 129.54 0))
     (pin "1")
@@
       (effects (font (size 1.27 1.27)) (justify right))
     )
-    (property "Footprint" "" (id 2) (at 132.08 111.76 0)
+    (property "Footprint" "kbd.pretty:D3_SMD" (id 2) (at 132.08 111.76 0)
       (effects (font (size 1.27 1.27)) hide)
     )
@@
       (effects (font (size 1.27 1.27)) (justify right))
     )
-    (property "Footprint" "" (id 2) (at 95.25 111.76 0)
+    (property "Footprint" "kbd.pretty:D3_SMD" (id 2) (at 95.25 111.76 0)
       (effects (font (size 1.27 1.27)) hide)
     )
@@
       (effects (font (size 1.27 1.27)) (justify right))
     )
-    (property "Footprint" "" (id 2) (at 95.25 133.35 0)
+    (property "Footprint" "kbd.pretty:D3_SMD" (id 2) (at 95.25 133.35 0)
       (effects (font (size 1.27 1.27)) hide)
     )
@@
     (property "Reference" "J2" (id 0) (at 40.132 50.165 0))
     (property "Value" "LED" (id 1) (at 40.132 52.4764 0))
-    (property "Footprint" "kbd:StripLED_rev" (id 2) (at 38.1 58.42 0)
+    (property "Footprint" "kbd.pretty:StripLED_rev" (id 2) (at 38.1 58.42 0)
       (effects (font (size 1.27 1.27)) hide)
     )
@@
     (property "Reference" "SW5" (id 0) (at 146.05 48.26 0))
     (property "Value" "SW_PUSH" (id 1) (at 146.05 50.8 0))
-    (property "Footprint" "" (id 2) (at 146.05 55.88 0))
+    (property "Footprint" "kbd.pretty:CherryMX_Choc_Hotswap" (id 2) (at 146.05 55.88 0)
+      (effects (font (size 1.27 1.27)) hide)
+    )
     (property "Datasheet" "" (id 3) (at 146.05 55.88 0))
     (pin "1")
@@
       (effects (font (size 1.524 1.524)))
     )
-    (property "Footprint" "" (id 2) (at 93.98 91.44 0)
-      (effects (font (size 1.524 1.524)))
+    (property "Footprint" "kbd.pretty:ProMicro_v2" (id 2) (at 93.98 91.44 0)
+      (effects (font (size 1.524 1.524)) hide)
     )
     (property "Datasheet" "" (id 3) (at 93.98 91.44 0)
@@
     )
     (path "/b8860185-f4b6-4df9-904a-e9c1bcaac6e5"
-      (reference "D1") (unit 1) (value "D") (footprint "")
+      (reference "D1") (unit 1) (value "D") (footprint "kbd.pretty:D3_SMD")
     )
     (path "/c6853e41-db12-4d94-9900-abcf4b21f196"
-      (reference "D2") (unit 1) (value "D") (footprint "")
+      (reference "D2") (unit 1) (value "D") (footprint "kbd.pretty:D3_SMD")
     )
     (path "/a6ee75b0-85a8-441d-90a3-484b20362429"
-      (reference "D3") (unit 1) (value "D") (footprint "")
+      (reference "D3") (unit 1) (value "D") (footprint "kbd.pretty:D3_SMD")
     )
     (path "/6d8f4292-68a9-48ad-94cb-10f853c18e7d"
-      (reference "D4") (unit 1) (value "D") (footprint "")
+      (reference "D4") (unit 1) (value "D") (footprint "kbd.pretty:D3_SMD")
     )
     (path "/6b3b531f-6c32-4eea-81f4-545457e20efe"
-      (reference "J1") (unit 1) (value "MJ-4PP-9") (footprint "")
+      (reference "J1") (unit 1) (value "MJ-4PP-9") (footprint "kbd.pretty:MJ-4PP-9")
     )
     (path "/fb4a35f3-6783-4dd7-8dfb-6a4cc6662230"
-      (reference "J2") (unit 1) (value "LED") (footprint "kbd:StripLED_rev")
+      (reference "J2") (unit 1) (value "LED") (footprint "kbd.pretty:StripLED_rev")
     )
     (path "/56060d9e-7b51-4fd5-8c53-acc51fc5f7a8"
-      (reference "SW1") (unit 1) (value "SW_PUSH") (footprint "")
+      (reference "SW1") (unit 1) (value "SW_PUSH") (footprint "kbd.pretty:CherryMX_Choc_Hotswap")
     )
     (path "/a4b12488-3c76-46b6-b0d1-fda5de7551e6"
-      (reference "SW2") (unit 1) (value "SW_PUSH") (footprint "")
+      (reference "SW2") (unit 1) (value "SW_PUSH") (footprint "kbd.pretty:CherryMX_Choc_Hotswap")
     )
     (path "/8f6593a8-66f1-4121-9086-420ba22ce8f5"
-      (reference "SW3") (unit 1) (value "SW_PUSH") (footprint "")
+      (reference "SW3") (unit 1) (value "SW_PUSH") (footprint "kbd.pretty:CherryMX_Choc_Hotswap")
     )
     (path "/3d7caea8-80eb-4571-bea4-80d198bd5d18"
-      (reference "SW4") (unit 1) (value "SW_PUSH") (footprint "")
+      (reference "SW4") (unit 1) (value "SW_PUSH") (footprint "kbd.pretty:CherryMX_Choc_Hotswap")
     )
     (path "/fe7812ac-aa19-41f6-9ed2-26e8d2611c1f"
-      (reference "SW5") (unit 1) (value "SW_PUSH") (footprint "")
+      (reference "SW5") (unit 1) (value "SW_PUSH") (footprint "kbd.pretty:CherryMX_Choc_Hotswap")
     )
     (path "/fff70b40-b639-4e03-b5d9-574111d4fa3d"
-      (reference "U1") (unit 1) (value "ProMicro") (footprint "")
-    )
-  )
+      (reference "U1") (unit 1) (value "ProMicro") (footprint "kbd.pretty:ProMicro_v2")
+    )
+  )

Commit message: complete PCB
Parts:
- SW5: value SW_PUSH -> RESET_SW; footprint kbd.pretty:CherryMX_Choc_Hotswap -> kbd.pretty:ResetSW
Changed lines of the file:
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@@
     (in_bom yes) (on_board yes) (fields_autoplaced)
     (property "Reference" "SW5" (id 0) (at 146.05 48.26 0))
-    (property "Value" "SW_PUSH" (id 1) (at 146.05 50.8 0))
-    (property "Footprint" "kbd.pretty:CherryMX_Choc_Hotswap" (id 2) (at 146.05 55.88 0)
+    (property "Value" "RESET_SW" (id 1) (at 146.05 50.8 0))
+    (property "Footprint" "kbd.pretty:ResetSW" (id 2) (at 146.05 55.88 0)
       (effects (font (size 1.27 1.27)) hide)
     )
@@
     )
     (path "/fe7812ac-aa19-41f6-9ed2-26e8d2611c1f"
-      (reference "SW5") (unit 1) (value "SW_PUSH") (footprint "kbd.pretty:CherryMX_Choc_Hotswap")
+      (reference "SW5") (unit 1) (value "RESET_SW") (footprint "kbd.pretty:ResetSW")
     )
     (path "/fff70b40-b639-4e03-b5d9-574111d4fa3d"
