File: KeyboardPlayer/KeyboardPlayer.kicad_pcb (KiCad board)
At the start: 2 copper layers, 67.2 x 67.2 mm, 16 parts, among them J1 MJ-4PP-9, J2 LED, SW1 SW_PUSH, SW2 RotaryEncoder_Switch, SW3 SW_PUSH, SW4 SW_PUSH, SW5 RESET_SW, SW6 SW_PUSH, SW7 SW_PUSH, U1 ProMicro

Commit message: add M2
Parts:
- added Ref**: Val**, kbd.pretty:HOLE, F.Cu at (33.0, 98.6)
- added Ref**: Val**, kbd.pretty:HOLE, F.Cu at (93.4, 139.8)
- added Ref**: Val**, kbd.pretty:HOLE, F.Cu at (33.0, 139.9)
- added Ref**: Val**, kbd.pretty:HOLE, F.Cu at (93.4, 98.6)
- moved J2 55.6 mm to (38.8, 136.7), turned to 0 degrees
Routing:
- net VCC: track 92.6 -> 135.2 mm, vias 2 -> 3
- net led-Din: track 56.6 -> 85.8 mm, vias 1 -> 2
- net GND: track 200.2 -> 184.6 mm
- net row-1: track 95.6 -> 93.1 mm

Commit message: paint GND
Routing:
- added copper zone on B.Cu, net GND
- added copper zone on F.Cu, net GND
Changed lines of the file:
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@@
   (segment (start 81.605504 78.972459) (end 81.605504 77.379499) (width 0.25) (layer "B.Cu") (net 28))
   (segment (start 82.875504 93.925899) (end 82.875504 80.242459) (width 0.25) (layer "B.Cu") (net 28))
+  (zone (net 12) (net_name "GND") (layers F&B.Cu) (hatch edge 0.508)
+    (connect_pads (clearance 0.508))
+    (min_thickness 0.254) (filled_areas_thickness no)
+    (fill yes (thermal_gap 0.508) (thermal_bridge_width 0.508))
+    (polygon
+      (pts
+        (xy 97.784004 144.219499)
+        (xy 28.784004 144.219499)
+        (xy 28.784004 75.219499)
+        (xy 97.784004 75.219499)
+      )
+    )
+  )
   (group "" (id 5a787f29-3dfa-44d3-8ad9-3da30c104885)
     (members

Commit message: finished version1.0
Parts:
- added REF**: SCK-logo, logo.pretty:SCK-logo, F.Cu at (41.0, 83.9)
Other:
- board text added: "Seekbar Control Keyboard PCB Designed by S.K."
