File: SeekbarControlKeyboard/pcb/SeekbarControlKeyboard.kicad_pcb (KiCad board)
At the start: 2 copper layers, 67.2 x 67.2 mm, 21 parts, among them J1 MJ-4PP-9, J2 LED, SW1 SW_PUSH, SW2 RotaryEncoder_Switch, SW3 SW_PUSH, SW4 SW_PUSH, SW5 RESET_SW, SW6 SW_PUSH, SW7 SW_PUSH, U1 ProMicro

Commit message: finished plate of bottom and top
Parts:
- moved J1 0.15 mm to (57.7, 76.2)
