File: pcb/SeekbarControlKeyboard.kicad_pcb (KiCad board)
At the start: 2 copper layers, 67.2 x 67.2 mm, 21 parts, among them J1 MJ-4PP-9, J2 LED, SW1 SW_PUSH, SW2 RotaryEncoder_Switch, SW3 SW_PUSH, SW4 SW_PUSH, SW5 RESET_SW, SW6 SW_PUSH, SW7 SW_PUSH, U1 ProMicro

Commit message: fix M2 PCB close #2
Parts:
- removed Ref** (x4): Val**, kbd.pretty:HOLE
- added REF**: M2_HOLE, kbd.pretty:M2_HOLE, F.Cu at (93.4, 98.6)
- added REF**: M2_HOLE, kbd.pretty:M2_HOLE, F.Cu at (33.0, 139.9)
- added REF**: M2_HOLE, kbd.pretty:M2_HOLE, F.Cu at (93.4, 139.8)
- added REF**: M2_HOLE, kbd.pretty:M2_HOLE, F.Cu at (33.0, 98.6)
Changed lines of the file:
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@@
     )
     (pad_to_mask_clearance 0)
-    (aux_axis_origin 40.834004 76.119499)
+    (aux_axis_origin 96.234004 96.949499)
     (grid_origin 96.784004 143.219499)
     (pcbplotparams
@@
   (net 27 "unconnected-(U1-Pad6)")
   (net 28 "unconnected-(U1-Pad5)")
+  (footprint "kbd.pretty:M2_HOLE" (layer "F.Cu")
+    (at 93.445504 98.604499)
+    (attr through_hole)
+    (fp_text reference "REF**" (at 0 -0.5 unlocked) (layer "F.SilkS") hide
+      (effects (font (size 1 1) (thickness 0.15)))
+    )
+    (fp_text value "M2_HOLE" (at 0 1.65 unlocked) (layer "F.Fab") hide
+      (effects (font (size 1 1) (thickness 0.15)))
+    )
+    (fp_text user "${REFERENCE}" (at 0 2.5 unlocked) (layer "F.Fab") hide
+      (effects (font (size 1 1) (thickness 0.15)))
+    )
+    (pad "1" thru_hole circle (at 0 0) (size 3 3) (drill 2.8) (layers *.Cu *.Mask))
+  )
   (footprint "kbd.pretty:D3_TH_SMD_v2" (layer "F.Cu")
     (at 87.157504 101.519499 180)
@@
       (net 5 "Net-(D3-Pad2)") (pinfunction "2") (pintype "passive"))
   )
-  (footprint "kbd.pretty:HOLE" (layer "F.Cu")
-    (at 33.033004 98.619499)
-    (descr "Mounting Hole 2.2mm, no annular, M2")
-    (tags "mounting hole 2.2mm no annular m2")
-    (attr exclude_from_pos_files exclude_from_bom)
-    (fp_text reference "Ref**" (at 0 -3.2) (layer "F.Fab")
-      (effects (font (size 1 1) (thickness 0.15)))
-    )
-    (fp_text value "Val**" (at 0 3.2) (layer "F.Fab")
-      (effects (font (size 1 1) (thickness 0.15)))
-    )
-    (fp_text user "${REFERENCE}" (at 0.3 0) (layer "F.Fab")
-      (effects (font (size 1 1) (thickness 0.15)))
-    )
-    (fp_circle (center 0 0) (end 2.2 0) (layer "Cmts.User") (width 0.15) (fill none))
-    (fp_circle (center 0 0) (end 2.45 0) (layer "F.CrtYd") (width 0.05) (fill none))
-    (pad "" np_thru_hole circle locked (at 0 0) (size 5 5) (drill 4.8) (layers *.Cu *.Mask))
-  )
   (footprint "kbd.pretty:D3_TH_SMD_v2" (layer "F.Cu")
     (at 87.157504 120.619499 180)
@@
       (rotate (xyz 0 0 0))
     )
-  )
-  (footprint "kbd.pretty:HOLE" (layer "F.Cu")
-    (at 93.384004 139.819499)
-    (descr "Mounting Hole 2.2mm, no annular, M2")
-    (tags "mounting hole 2.2mm no annular m2")
-    (attr exclude_from_pos_files exclude_from_bom)
-    (fp_text reference "Ref**" (at 0 -3.2) (layer "F.Fab")
-      (effects (font (size 1 1) (thickness 0.15)))
-    )
-    (fp_text value "Val**" (at 0 3.2) (layer "F.Fab")
-      (effects (font (size 1 1) (thickness 0.15)))
-    )
-    (fp_text user "${REFERENCE}" (at 0.3 0) (layer "F.Fab")
-      (effects (font (size 1 1) (thickness 0.15)))
-    )
-    (fp_circle (center 0 0) (end 2.2 0) (layer "Cmts.User") (width 0.15) (fill none))
-    (fp_circle (center 0 0) (end 2.45 0) (layer "F.CrtYd") (width 0.05) (fill none))
-    (pad "" np_thru_hole circle locked (at 0 0) (size 5 5) (drill 4.8) (layers *.Cu *.Mask))
   )
   (footprint "kbd.pretty:D3_TH_SMD_v2" (layer "F.Cu")
@@
       (net 7 "Net-(D5-Pad2)") (pinfunction "2") (pintype "passive"))
   )
+  (footprint "kbd.pretty:M2_HOLE" (layer "F.Cu")
+    (at 33.033004 139.896001)
+    (attr through_hole)
+    (fp_text reference "REF**" (at 0 -0.5 unlocked) (layer "F.SilkS") hide
+      (effects (font (size 1 1) (thickness 0.15)))
+    )
+    (fp_text value "M2_HOLE" (at 0 1.65 unlocked) (layer "F.Fab") hide
+      (effects (font (size 1 1) (thickness 0.15)))
+    )
+    (fp_text user "${REFERENCE}" (at 0 2.5 unlocked) (layer "F.Fab") hide
+      (effects (font (size 1 1) (thickness 0.15)))
+    )
+    (pad "1" thru_hole circle (at 0 0) (size 3 3) (drill 2.8) (layers *.Cu *.Mask))
+  )
   (footprint "kbd.pretty:D3_TH_SMD_v2" (layer "F.Cu")
     (at 68.157504 101.519499 180)
@@
       (rotate (xyz 0 0 0))
     )
-  )
-  (footprint "kbd.pretty:HOLE" (layer "F.Cu")
-    (at 33.033004 139.896001)
-    (descr "Mounting Hole 2.2mm, no annular, M2")
-    (tags "mounting hole 2.2mm no annular m2")
-    (attr exclude_from_pos_files exclude_from_bom)
-    (fp_text reference "Ref**" (at 0 -3.2) (layer "F.Fab")
-      (effects (font (size 1 1) (thickness 0.15)))
-    )
-    (fp_text value "Val**" (at 0 3.2) (layer "F.Fab")
-      (effects (font (size 1 1) (thickness 0.15)))
-    )
-    (fp_text user "${REFERENCE}" (at 0.3 0) (layer "F.Fab")
-      (effects (font (size 1 1) (thickness 0.15)))
-    )
-    (fp_circle (center 0 0) (end 2.2 0) (layer "Cmts.User") (width 0.15) (fill none))
-    (fp_circle (center 0 0) (end 2.45 0) (layer "F.CrtYd") (width 0.05) (fill none))
-    (pad "" np_thru_hole circle locked (at 0 0) (size 5 5) (drill 4.8) (layers *.Cu *.Mask))
   )
   (footprint "kbd.pretty:CherryMX_Choc_Hotswap" (layer "F.Cu")
@@
     (pad "2" smd rect (at 6.9 -2.54 180) (size 2 2) (layers "F.Cu" "F.Paste" "F.Mask")
       (net 2 "Net-(D1-Pad2)") (pinfunction "2") (pintype "passive"))
+  )
+  (footprint "kbd.pretty:M2_HOLE" (layer "F.Cu")
+    (at 93.384004 139.819499)
+    (attr through_hole)
+    (fp_text reference "REF**" (at 0 -0.5 unlocked) (layer "F.SilkS") hide
+      (effects (font (size 1 1) (thickness 0.15)))
+    )
+    (fp_text value "M2_HOLE" (at 0 1.65 unlocked) (layer "F.Fab") hide
+      (effects (font (size 1 1) (thickness 0.15)))
+    )
+    (fp_text user "${REFERENCE}" (at 0 2.5 unlocked) (layer "F.Fab") hide
+      (effects (font (size 1 1) (thickness 0.15)))
+    )
+    (pad "1" thru_hole circle (at 0 0) (size 3 3) (drill 2.8) (layers *.Cu *.Mask))
   )
   (footprint "kbd.pretty:StripLED_rev" (layer "F.Cu")
@@
     )
   )
-  (footprint "kbd.pretty:HOLE" (layer "F.Cu")
-    (at 93.445504 98.604499)
-    (descr "Mounting Hole 2.2mm, no annular, M2")
-    (tags "mounting hole 2.2mm no annular m2")
-    (attr exclude_from_pos_files exclude_from_bom)
-    (fp_text reference "Ref**" (at 0 -3.2) (layer "F.Fab")
-      (effects (font (size 1 1) (thickness 0.15)))
-    )
-    (fp_text value "Val**" (at 0 3.2) (layer "F.Fab")
-      (effects (font (size 1 1) (thickness 0.15)))
-    )
-    (fp_text user "${REFERENCE}" (at 0.3 0) (layer "F.Fab")
-      (effects (font (size 1 1) (thickness 0.15)))
-    )
-    (fp_circle (center 0 0) (end 2.2 0) (layer "Cmts.User") (width 0.15) (fill none))
-    (fp_circle (center 0 0) (end 2.45 0) (layer "F.CrtYd") (width 0.05) (fill none))
-    (pad "" np_thru_hole circle locked (at 0 0) (size 5 5) (drill 4.8) (layers *.Cu *.Mask))
-  )
   (footprint "Keebio-Parts.pretty:RotaryEncoder_EC11" (layer "F.Cu")
     (at 44.157504 128.769499)
@@
     )
   )
+  (footprint "kbd.pretty:M2_HOLE" (layer "F.Cu")
+    (at 33.033004 98.619499)
+    (attr through_hole)
+    (fp_text reference "REF**" (at 0 -0.5 unlocked) (layer "F.SilkS") hide
+      (effects (font (size 1 1) (thickness 0.15)))
+    )
+    (fp_text value "M2_HOLE" (at 0 1.65 unlocked) (layer "F.Fab") hide
+      (effects (font (size 1 1) (thickness 0.15)))
+    )
+    (fp_text user "${REFERENCE}" (at 0 2.5 unlocked) (layer "F.Fab") hide
+      (effects (font (size 1 1) (thickness 0.15)))
+    )
+    (pad "1" thru_hole circle (at 0 0) (size 3 3) (drill 2.8) (layers *.Cu *.Mask))
+  )
   (gr_line (start 93.225974 95.195) (end 99.633004 95.195) (layer "Dwgs.User") (width 0.15))

Commit message: exchange rotary encoder and switch
Parts:
- moved SW1 19.0 mm to (44.2, 128.8)
- moved SW2 19.0 mm to (44.2, 109.7)
Connections:
- SW1 pad 2: Net-(D1-Pad2) -> Net-(D2-Pad2)
- SW2 pad S1: Net-(D2-Pad2) -> Net-(D1-Pad2)
Routing:
- net rotary-A: track 79.7 -> 59.3 mm
- net Net-(D2-Pad2): track 13.3 -> 27.1 mm, vias 0 -> 2
- net Net-(D1-Pad2): track 25.6 -> 14.0 mm, vias 2 -> 0
- net rotary-B: track 83.7 -> 73.4 mm
- net GND: track 184.7 -> 178.4 mm, vias 3 -> 2
- net VCC: track 135.0 -> 131.2 mm
- net col-0: track 108.6 -> 106.2 mm, vias 1 -> 2
- net led-Din: track 85.8 -> 84.5 mm, vias 2 -> 1

Commit message: move folder and fix Diode fotprint close #4
Parts:
- D1, D2, D3, D4, D5, D6: footprint kbd.pretty:D3_TH_SMD_v2 -> parts:D3_TH_SMD_v3
Routing:
- net row-1: track 93.1 -> 95.6 mm
